Commit message: Update correct package name and included three new tf to urdf.

File: robots/fetch.gazebo.xacro (robot description, xacro)
@@ -1,4 +1,4 @@
 <robot xmlns:xacro="http://www.ros.org/wiki/xacro" name="fetch" >
-  <xacro:include filename="$(find fetch_sim2real)/robots/fetch.urdf" />
+  <xacro:include filename="$(find uv_project)/robots/fetch.urdf" />
   <!-- Add four casters to the base -->
   <xacro:macro name="caster" params="prefix joint_x joint_y">

File: robots/fetch.urdf (robot description, URDF)
Before this commit: robot fetch, 27 links, 26 joints
Links:
- removed link ee_link
- added link camera_color_optical_frame
- added link camera_link
- added link uv_light_link
Joints:
- removed joint ee_joint
- added joint camera_color_optical_frame_joint: type fixed, parent camera_link, child camera_color_optical_frame, origin xyz=-0.0003675 0.014825 0.00014789 rpy=-1.5707963267948968 0.0 -1.5707963267948968, axis 0 0 0
- added joint camera_joint: type fixed, parent gripper_link, child camera_link, origin xyz=-0.09 0.0175 -0.063 rpy=0 1.57079632679 0, axis 0 0 0
- added joint uv_light_joint: type fixed, parent gripper_link, child uv_light_link, origin xyz=0 0 -0.08 rpy=0 0 0, axis 0 0 0
